File: eagle/tf536.brd (EAGLE design)
At the start: 104.1 x 100.6 mm, 74 parts, among them IC1 MC68030, IC10 74VHC245PW,118, IC2 LM1117-3.3, IC3 SAMACSYS_PARTS_XC95144XL-10TQ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, IC4 74VHC245PW,118, IC5 74VHC245PW,118, IC6 74VHC245PW,118, IC7 MT48LC16M16A2P-6A_G, IC8 MT48LC16M16A2P-6A_G, IC9 74VHC245PW,118, U1 SN74CB3T3245PW, U2 SN74CB3T3245PW, U3 SN74CB3T3245PW, U4 SN74CB3T3245PW, X1 MC68000

Commit message: Updating the schematic to say XC95288XL
Parts:
- IC3: value SAMACSYS_PARTS_XC95144XL-10TQG144I -> XC95288XL-10TQG144I
Changed lines of the file:
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@@
 <attribute name="PRICE" value="None" x="98.4758" y="47.2948" size="1.778" layer="27" rot="R90" display="off"/>
 </element>
-<element name="IC3" library="sjl540" package="SAMACSYS_PARTS_QFP50P2200X2200X160-144N" value="SAMACSYS_PARTS_XC95144XL-10TQG144I" x="48.5394" y="68.2244" smashed="yes" rot="R225">
+<element name="IC3" library="sjl540" package="SAMACSYS_PARTS_QFP50P2200X2200X160-144N" value="XC95288XL-10TQG144I" x="48.5394" y="68.2244" smashed="yes" rot="R225">
 <attribute name="3D_PACKAGE" value="" x="48.5394" y="68.2244" size="1.778" layer="27" rot="R225" display="off"/>
 <attribute name="DESCRIPTION" value="XC95144XL-10TQG144I XC95144XL-10TQG144I, CPLD XC9500XL Flash 144 Cells, 117 I/O, 8 Labs, ISP, 3  3.6 V 144-Pin TQFP" x="48.5394" y="68.2244" size="1.778" layer="27" rot="R225" display="off"/>

Commit message: Add Eagle netlist and UCF generation tools
- Add generate_netlist.py to export Eagle schematic to netlist format
- Add generate_ucf.py to generate UCF files from Eagle netlists
  - Filters power (GND, VCC) and JTAG (TCK/TDI/TDO/TMS) signals
  - Handles 68030-specific signals (AS30, BG30, etc.) correctly
  - Optional --remap-dbus flag to map D16-D31 to D<0>-D<15>
- Update Eagle schematic signal names to match UCF conventions:
  - CLK7M -> CLK7M_RAW
  - DS30ACK0/1 -> DSACK0/1
  - Fix DQM0-3 pin mapping
Connections:
- net CLK7M renamed CLK7M_RAW
- net DS30ACK0 renamed DSACK0
- net DS30ACK1 renamed DSACK1
- net DQM0: now also IC3.3, IC7.39; no longer IC3.16, IC8.15
- net DQM1: now also IC3.15, IC7.15; no longer IC3.31, IC8.39
- net DQM2: now also IC3.31, IC8.39; no longer IC3.15, IC7.15
- net DQM3: now also IC3.16, IC8.15; no longer IC3.3, IC7.39
Routing:
- net DQM3: track 12.1 -> 55.1 mm
- net DQM0: track 55.1 -> 12.1 mm
- net DQM2: track 31.2 -> 57.5 mm
- net DQM1: track 57.5 -> 31.2 mm
Changed lines of the file:
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@@
 <wire x1="41.4909" y1="51.629959375" x2="41.4909" y2="30.7467" width="0.1524" layer="1"/>
 </signal>
-<signal name="DQM3">
+<signal name="DQM0">
 <contactref element="IC7" pad="39"/>
 <contactref element="IC3" pad="3"/>
@@
 <wire x1="66.770425" y1="68.0972" x2="72.1738" y2="68.0972" width="0.1524" layer="1"/>
 </signal>
-<signal name="DQM2">
+<signal name="DQM1">
 <contactref element="IC7" pad="15"/>
 <contactref element="IC3" pad="15"/>
@@
 <wire x1="59.701071875" y1="76.9112" x2="69.6722" y2="76.9112" width="0.1524" layer="1"/>
 </signal>
-<signal name="DQM1">
+<signal name="DQM2">
 <contactref element="IC8" pad="39"/>
 <contactref element="IC3" pad="31"/>
@@
 <wire x1="51.71289375" y1="80.236728125" x2="61.912865625" y2="90.4367" width="0.1524" layer="1"/>
 </signal>
-<signal name="DQM0">
+<signal name="DQM3">
 <contactref element="IC8" pad="15"/>
 <wire x1="101.4606" y1="77.5588" x2="100.6476" y2="77.5588" width="0.1524" layer="1"/>
@@
 <wire x1="60.187765625" y1="78.105" x2="73.7108" y2="78.105" width="0.1524" layer="1"/>
 </signal>
-<signal name="DS30ACK1">
+<signal name="DSACK1">
 <contactref element="IC1" pad="G02"/>
 <contactref element="IC3" pad="92"/>
@@
 <wire x1="48.62694375" y1="16.87694375" x2="50.32874375" y2="16.87694375" width="0.1524" layer="1"/>
 </signal>
-<signal name="DS30ACK0">
+<signal name="DSACK0">
 <contactref element="IC1" pad="F01"/>
 <contactref element="IC3" pad="93"/>
@@
 <wire x1="13.705" y1="28.459" x2="5.6896" y2="36.4744" width="0.1524" layer="16"/>
 </signal>
-<signal name="CLK7M">
+<signal name="CLK7M_RAW">
 <contactref element="X1" pad="15"/>
 <contactref element="IC3" pad="66"/>
